File: uMotion_v1.0.sch (EAGLE design)
At the start: 130 parts, among them IC1 LM1117-3.3, IC2 LM4040B25, IC3 LM1117-3.3, IC4 DAC8552, IC5 TL072, IC6 TL072, IC7 LM4040B10, IC8 MCP6002, IC9 MCP6004, J1 WQP-PJ301M-12_JACK, J10 WQP-PJ301M-12_JACK, J11 WQP-PJ301M-12_JACK, J12 WQP-PJ301M-12_JACK, J13 WQP-PJ301M-12_JACK, J2 WQP-PJ301M-12_JACK, J3 WQP-PJ301M-12_JACK, J4 WQP-PJ301M-12_JACK, J5 WQP-PJ301M-12_JACK, J6 WQP-PJ301M-12_JACK, J7 WQP-PJ301M-12_JACK, J8 WQP-PJ301M-12_JACK, J9 WQP-PJ301M-12_JACK, Q1 8MHz, Q2 MMBT3904, Q3 MMBT3904, Q4 MMBT3904, Q5 MMBT3904, Q6 MMBT3904

Commit message: uMotion files
Other:
- note added: "Codex-Modulex"
- note added: "Original design by: Olivier Gillet of Mutable Instruments"
- note added: "info@codex-modulex.com"
- note removed: "Olivier Gillet"
- note removed: "ol.gillet@gmail.com"
